File: ejemplos/KiCad/src/E-Textil/Big_4_Pin/001.kicad_pcb (KiCad board)
At the start: 2 copper layers, 22.8 x 45 mm, 14 parts, among them J2 CONN_01X01, J4 CONN_01X01, J5 CONN_01X01, J6 CONN_01X01

Commit message: Update Repo 04.04.19 (#1)
* Update README.md

* Create README.md

* Create prueba.txt

* Add files via upload

* Delete prueba.txt

* Update README.md

* Create prueba.txt

* Add files via upload

* Delete prueba.txt

* Update README.md

* Update README.md

* Update README.md

* Documentación proyecto

Modificado el Readme.md del proyecto, añadido fotos y mejorar del código
con comentarios.

* Update README.md

* Rename semaforo_NeoPixel16LED.py to main.py

* Update README.md

* Update README.md

* Corregida ruta imágenes

Corregida ruta imágenes

* Add files via upload

* Add files via upload

* Create Node-RED

* Delete Node-RED

* Add files via upload

* Create README.md

* Add files via upload

* Update README.md

* Update README.md

* Create Formatted JSON flows

* Create Compact JSON flows

* Update README.md

* Update README.md

* Add files via upload

* Delete Compact JSON flows

* Delete Formatted JSON flows

* Update README.md

* Add Universal PCB 10mm Semaforo

* Ejemplo Esp8266 con Thingerio

* Update README.md

* Add PCB for 555 and Atiny85

* Blender 3D

* Add Makecode example

:v

* Update Readme.md

* Nuevas imagenes

* Add files via upload

* Create README.md

* Create Readme.md

* Create Readme.md

* Add files via upload

* Update Readme.md

* Update Readme.md

* Update Readme.md

* Delete cp10.jpg

* Delete cp11.jpg

* Update Readme.md

* Update Readme.md

* Update Readme.md

* Add files via upload

* Update Readme.md

* Update Readme.md

* correccion carpeta

* correccion carpeta

* Create README.md

* Add files via upload

* Delete Image-1.jpg

* Delete Image-2.jpg

* Delete Image-3.jpg

* Delete Semaforo-icestudio.png

* Auto stash before merge of "master" and "origin/master"

* Add Universal 4 Pin PCB

* Update Readme in Kicad

* Update Readme in parent new PCB Universal

* Some minors updates

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
Parts:
- removed G***: LOGO, OshPark_Version:greynaga6-2
- removed GS***: v, OshPark_Version:greynaga6-2-cooper
- added svg2mod: G***, Universal:Developed-Silks3, B.Cu at (139.6, 118.9)
- added svg2mod: G***, Universal:GReynaga.CuMask3, B.Cu at (139.5, 127.6)
Routing:
- net Net-(D3-Pad2): track 17.6 -> 21.0 mm
- net Net-(D2-Pad2): track 23.9 -> 27.1 mm
- net Net-(D1-Pad2): track 25.3 -> 24.6 mm, vias 0 -> 2
- net GND: vias 4 -> 5
Other:
- board text removed: "Design By:"
