File: ejemplos/KiCad/src/E-Textil/Mini_6_Pin/001.kicad_pcb (KiCad board)
At the start: 2 copper layers, 22.8 x 26.9 mm, 13 parts, among them J1 CONN_01X01, J2 CONN_01X01, J3 CONN_01X01, J4 CONN_01X01, J5 CONN_01X01, J6 CONN_01X01

Commit message: Update Repo 04.04.19 (#1)
* Update README.md

* Create README.md

* Create prueba.txt

* Add files via upload

* Delete prueba.txt

* Update README.md

* Create prueba.txt

* Add files via upload

* Delete prueba.txt

* Update README.md

* Update README.md

* Update README.md

* Documentación proyecto

Modificado el Readme.md del proyecto, añadido fotos y mejorar del código
con comentarios.

* Update README.md

* Rename semaforo_NeoPixel16LED.py to main.py

* Update README.md

* Update README.md

* Corregida ruta imágenes

Corregida ruta imágenes

* Add files via upload

* Add files via upload

* Create Node-RED

* Delete Node-RED

* Add files via upload

* Create README.md

* Add files via upload

* Update README.md

* Update README.md

* Create Formatted JSON flows

* Create Compact JSON flows

* Update README.md

* Update README.md

* Add files via upload

* Delete Compact JSON flows

* Delete Formatted JSON flows

* Update README.md

* Add Universal PCB 10mm Semaforo

* Ejemplo Esp8266 con Thingerio

* Update README.md

* Add PCB for 555 and Atiny85

* Blender 3D

* Add Makecode example

:v

* Update Readme.md

* Nuevas imagenes

* Add files via upload

* Create README.md

* Create Readme.md

* Create Readme.md

* Add files via upload

* Update Readme.md

* Update Readme.md

* Update Readme.md

* Delete cp10.jpg

* Delete cp11.jpg

* Update Readme.md

* Update Readme.md

* Update Readme.md

* Add files via upload

* Update Readme.md

* Update Readme.md

* correccion carpeta

* correccion carpeta

* Create README.md

* Add files via upload

* Delete Image-1.jpg

* Delete Image-2.jpg

* Delete Image-3.jpg

* Delete Semaforo-icestudio.png

* Auto stash before merge of "master" and "origin/master"

* Add Universal 4 Pin PCB

* Update Readme in Kicad

* Update Readme in parent new PCB Universal

* Some minors updates

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
Parts:
- added svg2mod: G***, Universal:Developed-Silks3, B.Cu at (139.4, 113.4)
- added svg2mod: G***, Universal:GReynaga.CuMask3, B.Cu at (138.6, 114.8)
- renumbered D3 to GREEN, D1 to RED, D2 to YELLOW
Routing:
- net Net-(D3-Pad2): track 6.79 -> 8.24 mm
- net Net-(D2-Pad2): track 6.63 -> 7.93 mm
- net Net-(D1-Pad2): track 6.78 -> 8.05 mm
Other:
- board text added: "v1.0"
- board text removed: "Design By"
- board text removed: "v 1.0"
